File: hardware/transmitter/transmitter.kicad_sch (KiCad schematic)
At the start: 27 parts, among them J1 Conn_01x05_Male, J2 Conn_01x05_Male, J3 Conn_02x08_Odd_Even, J4 Conn_02x04_Odd_Even, SW1 SW_Push_Dual, U1 ATmega328P-P, U2 MCP1700-3302E_SOT23, Y1 16MHz

Commit message: hardware transmitter: 200R
Parts:
- R1, R2, R3, R4: value 100R -> 200R
Changed lines of the file:
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@@
     (in_bom yes) (on_board yes)
     (property "Reference" "R4" (id 0) (at 107.95 95.25 90))
-    (property "Value" "100R" (id 1) (at 107.95 97.79 90))
+    (property "Value" "200R" (id 1) (at 107.95 97.79 90))
     (property "Footprint" "" (id 2) (at 107.95 94.488 90)
       (effects (font (size 1.27 1.27)) hide)
@@
     (in_bom yes) (on_board yes)
     (property "Reference" "R2" (id 0) (at 107.95 76.2 90))
-    (property "Value" "100R" (id 1) (at 107.95 78.74 90))
+    (property "Value" "200R" (id 1) (at 107.95 78.74 90))
     (property "Footprint" "" (id 2) (at 107.95 75.438 90)
       (effects (font (size 1.27 1.27)) hide)
@@
     (in_bom yes) (on_board yes) (fields_autoplaced)
     (property "Reference" "R3" (id 0) (at 115.57 83.82 90))
-    (property "Value" "100R" (id 1) (at 115.57 86.36 90))
+    (property "Value" "200R" (id 1) (at 115.57 86.36 90))
     (property "Footprint" "" (id 2) (at 115.57 91.948 90)
       (effects (font (size 1.27 1.27)) hide)
@@
     (in_bom yes) (on_board yes) (fields_autoplaced)
     (property "Reference" "R1" (id 0) (at 115.57 64.77 90))
-    (property "Value" "100R" (id 1) (at 115.57 67.31 90))
+    (property "Value" "200R" (id 1) (at 115.57 67.31 90))
     (property "Footprint" "" (id 2) (at 115.57 72.898 90)
       (effects (font (size 1.27 1.27)) hide)
@@
     )
     (path "/ffeba967-87d5-4070-b68e-66cb779b36e3"
-      (reference "R1") (unit 1) (value "100R") (footprint "")
+      (reference "R1") (unit 1) (value "200R") (footprint "")
     )
     (path "/8f65a448-d676-4d4e-b27a-255a02deec58"
-      (reference "R2") (unit 1) (value "100R") (footprint "")
+      (reference "R2") (unit 1) (value "200R") (footprint "")
     )
     (path "/b535f9f9-76b8-482f-b236-7d49c905253d"
-      (reference "R3") (unit 1) (value "100R") (footprint "")
+      (reference "R3") (unit 1) (value "200R") (footprint "")
     )
     (path "/7dd61320-2d42-4c02-b54e-4a2b1d08ec13"
-      (reference "R4") (unit 1) (value "100R") (footprint "")
+      (reference "R4") (unit 1) (value "200R") (footprint "")
     )
     (path "/293af796-5531-45ee-95f7-52c41e1e8a8f"
